Commit message: Add README, demo video, docs and full project

File: src/nav_robot_description/urdf/nav_robot.urdf (robot description, URDF)
Before this commit: robot nav_robot, 7 links, 6 joints
Links:
- added link camera_link, mass 0.05; visual box size=0.08 0.05 0.04
Joints:
- added joint camera_joint: type fixed, parent base_link, child camera_link, origin xyz=0.25 0 0.25 rpy=-1.5708 0 -1.5708
